File: control.brd (EAGLE design)
At the start: 100 x 50 mm, 12 parts, among them IC1 74AUC1G06DBV, IC2 74AHC1G32DBV

Commit message: opcode validator circuit thingy
Parts:
- added JP2: (no value), pinhead:1X08
Connections:
- new net IR1: JP2.8
- new net IR2: JP2.7
- new net IR3: JP2.6
- new net IR4: JP2.5
- new net IR5: JP2.4
- new net IR6: JP2.3
- new net IR7: JP2.2
- new net IR8: JP2.1
Changed lines of the file:
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@@
 <setting verticaltext="up"/>
 </settings>
-<grid distance="10" unitdist="mm" unit="mm" style="lines" multiple="1" display="yes" altdistance="5" altunitdist="mil" altunit="mil"/>
+<grid distance="12.5" unitdist="mil" unit="mil" style="lines" multiple="1" display="yes" altdistance="5" altunitdist="mil" altunit="mil"/>
 <layers>
 <layer number="1" name="Top" color="4" fill="1" visible="yes" active="yes"/>
@@
 <attribute name="VALUE" x="8.255" y="50.165" size="1.27" layer="27" rot="R180"/>
 </element>
+<element name="JP2" library="pinhead" library_urn="urn:adsk.eagle:library:325" package="1X08" package3d_urn="urn:adsk.eagle:package:22409/2" value="" x="81.28" y="4.7625" smashed="yes" rot="R180">
+<attribute name="NAME" x="91.5162" y="2.9337" size="1.27" layer="25" ratio="10" rot="R180"/>
+<attribute name="POPULARITY" value="67" x="81.28" y="4.7625" size="1.778" layer="27" rot="R180" display="off"/>
+<attribute name="VALUE" x="91.44" y="7.9375" size="1.27" layer="27" rot="R180"/>
+</element>
 </elements>
 <signals>
@@
 <wire x1="8.255" y1="48.26" x2="8.37" y2="48.26" width="0.1524" layer="1"/>
 </signal>
+<signal name="IR1">
+<contactref element="JP2" pad="8"/>
+</signal>
+<signal name="IR2">
+<contactref element="JP2" pad="7"/>
+</signal>
+<signal name="IR3">
+<contactref element="JP2" pad="6"/>
+</signal>
+<signal name="IR4">
+<contactref element="JP2" pad="5"/>
+</signal>
+<signal name="IR5">
+<contactref element="JP2" pad="4"/>
+</signal>
+<signal name="IR6">
+<contactref element="JP2" pad="3"/>
+</signal>
+<signal name="IR7">
+<contactref element="JP2" pad="2"/>
+</signal>
+<signal name="IR8">
+<contactref element="JP2" pad="1"/>
+</signal>
 </signals>
