File: ir_validator.brd (EAGLE design)
At the start: 70 x 60 mm, 27 parts, among them IC1 74LS688DW, IC10 74LS688DW, IC11 74AHC1G08DBV, IC12 74AHC1G04DBV, IC13 74LS688DW, IC14 74AHC1G08DBV, IC15 74AHC1G04DBV, IC16 74LS688DW, IC17 74AHC1G08DBV, IC18 74AHC1G04DBV, IC19 74LS688DW, IC2 74AHC1G08DBV, IC20 74AHC1G08DBV, IC21 74AHC1G04DBV, IC22 74LS688DW, IC23 74AHC1G08DBV, IC24 74AHC1G04DBV, IC3 74AHC1G04DBV, IC4 74LS688DW, IC5 74AHC1G08DBV, IC6 74AHC1G04DBV, IC7 74LS688DW, IC8 74AHC1G08DBV, IC9 74AHC1G04DBV

Commit message: some work
Parts:
- added IC25: 74LS688DW, 74xx-us:SO20W
- added IC26: 74AHC1G04DBV, 74xx-little-us:SOT23-5
- moved JP1 2.54 mm to (15.2, 2.54)
- moved JP2 2.54 mm to (36.8, 2.54)
- moved JP3 2.54 mm to (50.8, 2.54)
Connections:
- new net N$1: IC25.19, IC26.2
- net A2: now also IC25.2
- net B2: now also IC25.4
- net C2: now also IC25.6
- net D2: now also IC25.8
- net E2: now also IC25.11
- net F2: now also IC25.13
- net G2: now also IC25.15
- net GND: now also IC25.1, IC25.10, IC25.12, IC25.14, IC25.16, IC25.18, IC25.3, IC25.5, IC25.7, IC25.9, IC26.3
- net H2: now also IC25.17
- net HALT: now also IC26.4
- net VCC: now also IC25.20, IC26.5
Routing:
- net GND: track 415.9 -> 567.0 mm
- net A2: track 41.9 -> 87.3 mm, vias 1 -> 3
- net C: track 130.5 -> 175.0 mm, vias 4 -> 7
- net F2: track 54.6 -> 96.7 mm, vias 1 -> 2
- net B2: track 25.9 -> 66.6 mm, vias 1 -> 2
- net A: track 187.1 -> 146.8 mm, vias 9 -> 8
- net D2: track 36.4 -> 75.4 mm
- net B: track 182.5 -> 145.8 mm, vias 4 -> 7
- net C2: track 21.1 -> 56.7 mm, vias 1 -> 2
- net F: track 190.1 -> 164.3 mm
- net G2: track 41.7 -> 64.8 mm, vias 1 -> 2
- net VCC: track 278.6 -> 296.7 mm
- net E: track 185.4 -> 201.7 mm, vias 11 -> 10
- net HALT: track 0.00 -> 11.8 mm
- net N$1: track 0.00 -> 7.98 mm
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Other:
- board size 70 x 60 mm -> 69 x 49.2 mm
