File: register.brd (EAGLE design)
At the start: 100.3 x 74.9 mm, 64 parts, among them IC1 D(574), IC10 AND(08), IC2 D(574), IC3 ADD(283), IC4 ADD(283), IC5 ADD(283), IC6 ADD(283), IC7 BUF(244), IC8 BUF(244), IC9 NOT(04)

Commit message: add gerbers
Parts:
- added C1, C2, C3, C4, C5: C-Decouple, rcl:C025-025X050
- added H1, H2, H3: MOUNT-HOLE3.0, holes:3,0
- moved IC3 0.28 mm to (23.2, 33.0), turned to 180 degrees
- moved IC4 0.06 mm to (44.4, 33.0), turned to 180 degrees
Connections:
- net GND: now also C1.2, C2.2, C3.2, C4.2, C5.2
- net VCC: now also C1.1, C2.1, C3.1, C4.1, C5.1
Routing:
- net GND: track 257.6 -> 373.9 mm, vias 2 -> 1
- net Z: track 77.1 -> 190.9 mm, vias 1 -> 0
- net Q14: track 65.9 -> 166.0 mm, vias 2 -> 0
- net INC: track 104.0 -> 195.5 mm, vias 3 -> 5
- net Q8: track 112.3 -> 71.8 mm
- net N$4: track 103.0 -> 140.9 mm, vias 0 -> 1
- net B7: track 132.3 -> 96.3 mm, vias 2 -> 1
- net N$16: track 7.03 -> 36.6 mm
- net RD: track 97.8 -> 127.1 mm, vias 1 -> 6
- net CLK: track 105.9 -> 135.0 mm, vias 2 -> 6
- net B4: track 108.8 -> 80.0 mm, vias 1 -> 2
- net VCC: track 254.1 -> 282.2 mm, vias 2 -> 3
- net N$25: track 26.5 -> 4.48 mm
- net B8: track 64.8 -> 86.7 mm, vias 2 -> 0
- net B13: track 74.9 -> 54.7 mm, vias 1 -> 0
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Other:
- outline, holes or cut-outs redrawn

Commit message: rearrange
Parts:
- moved C5 78.2 mm to (94.0, 25.4), turned to 180 degrees
- moved JP4 35.8 mm to (68.6, 8.89)
- moved R10 35.3 mm to (62.2, 15.9)
- moved R11 35.3 mm to (64.8, 15.9)
- moved R12 35.3 mm to (67.3, 15.9)
- moved R13 35.3 mm to (69.8, 15.9)
- moved R14 35.3 mm to (72.4, 15.9)
- moved R16 35.3 mm to (77.5, 15.9)
- moved R9 35.3 mm to (59.7, 15.9)
- moved R15 35.3 mm to (74.9, 15.9)
- moved JP3 30.8 mm to (43.2, 8.89)
- moved R1 30.5 mm to (34.3, 15.9)
- moved R2 30.5 mm to (36.8, 15.9)
- moved R3 30.5 mm to (39.4, 15.9)
- moved R4 30.5 mm to (41.9, 15.9)
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Routing:
- net Z: track 190.9 -> 70.7 mm, vias 0 -> 5
- net WE: track 120.1 -> 205.8 mm
- net Q15: track 74.2 -> 159.5 mm, vias 0 -> 2
- net CLK2: track 114.0 -> 197.6 mm
- net Q13: track 67.8 -> 150.9 mm
- net B11: track 109.5 -> 38.5 mm, vias 1 -> 0
- net B6: track 114.8 -> 47.6 mm, vias 3 -> 0
- net RD: track 127.1 -> 185.3 mm, vias 6 -> 2
- net VCC: track 282.2 -> 337.2 mm, vias 3 -> 2
- net B1: track 107.4 -> 55.0 mm, vias 7 -> 1
- net Q3: track 47.4 -> 97.6 mm, vias 0 -> 2
- net N$4: track 140.9 -> 91.6 mm, vias 1 -> 0
- net B8: track 86.7 -> 37.5 mm
- net Q14: track 166.0 -> 120.3 mm, vias 0 -> 3
- net Q5: track 44.4 -> 89.1 mm
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Other:
- outline, holes or cut-outs redrawn
